File: Hardware/Kicad/audio_pwr_amp_r3.kicad_sch (KiCad schematic)
At the start: 58 parts, among them J1 Audio Out, J2 Audio Output, J3 INPUT_PWR, Q1 DMG2301L, U1 LM1875, U2 PTN78000AAH

Commit message: Add files via upload
Parts:
- removed C20: 10uF, Capacitor_SMD:C_0805_2012Metric_Pad1.18x1.45mm_HandSolder, symbol Device:C_Small
- removed C8: 22uF, Capacitor_SMD:C_1206_3216Metric_Pad1.33x1.80mm_HandSolder, symbol Device:C_Polarized_Small_US
- added C17: 10uF, Capacitor_SMD:C_0805_2012Metric_Pad1.18x1.45mm_HandSolder, symbol Device:C_Small
- added C8: 22uF, Capacitor_SMD:C_0805_2012Metric_Pad1.18x1.45mm_HandSolder, symbol Device:C_Small
- C1, C12, C15, C5: Vendor (none) -> Digikey; Vendor Part# (none) -> 399-A750MV108M1EAAE014-ND
- C10, C18, C19, C21, C22: Vendor # 1276-1017-1-ND -> (none); Vendor Part# (none) -> 1276-1099-1-ND
- C11, C13, C14: Vendor # 1276-1017-1-ND -> (none); Vendor Part# (none) -> 1276-1244-1-ND
- C16, C2, C3, C6: Vendor # 1276-1017-1-ND -> (none); Vendor Part# (none) -> 1276-6454-1-ND
- C4: Vendor # 1276-1017-1-ND -> (none); Vendor Part# (none) -> 399-14402-1-ND
- C7: value 100pF -> DNL; Vendor # 1276-1017-1-ND -> (none); now left out of the parts list
- C9: Vendor # 1276-1017-1-ND -> (none); Vendor Part# (none) -> 1276-1161-1-ND
- D1, D2: value OC_Fault -> RED_LED; Vendor Part # 1497-XZM2CRK55W-3RTCT-ND -> (none); Vendor Part# (none) -> 1497-XZM2CRK55W-3RTCT-ND
- FB1, FB2: value FerriteBead, 6A 1 9mΩ 33Ω@100MHz ±25% 1206 Ferrite Beads ROHS -> FERRITE CORE SOLID 1.30MM; Vendor Part # 1934-1465-1-ND -> (none); Vendor Part# (none) -> 1934-1292-ND
- H1, H2, H3, H4: now left out of the parts list
- J1: value Audio Out -> Audio In; Vendor (none) -> Digikey; Vendor Part# (none) -> CP-3524SJBECT-ND
- J2: LCSC No Stock -> (none); Vendor (none) -> Digikey; Vendor Part# (none) -> ED2609-ND
- J3: Vendor Part # CP-037A-ND -> (none); Vendor Part# (none) -> CP-037A-ND
- Q1: Vendor (none) -> Digikey; Vendor Part# (none) -> DMG2301L-7DICT-ND
- R1, R3: Vendor (none) -> Digikey; Vendor Part# (none) -> RMCF0805FT100RCT-ND
- R10: Vendor (none) -> Digikey; Vendor Part# (none) -> 311-100KCRCT-ND
- R11, R14, R9: Vendor (none) -> Digikey; Vendor Part# (none) -> 311-10.0KCRCT-ND
- R12: Vendor (none) -> Digikey; Vendor Part# (none) -> P2.00KCCT-ND
- R13, R8: Vendor (none) -> Digikey; Vendor Part# (none) -> 311-1.00KCRCT-ND
- R2: Vendor (none) -> Digikey; Vendor Part# (none) -> 311-0.0ARCT-ND
- R5, R6: Vendor (none) -> Digikey; Vendor Part# (none) -> P20KDACT-ND
- R7: Vendor (none) -> Digikey; Vendor Part# (none) -> 541-1.00TCT-ND
- RV1: value 5k -> 1k; Vendor # 987-1177-ND -> (none); Vendor Part# (none) -> 3386F-1-102TLF-ND
- U1: Vendor (none) -> Digikey; Vendor Part# (none) -> LM1875T/NOPB-ND
- U2: Vendor (none) -> Digikey; Vendor Part# (none) -> 296-20501-ND
Connections:
- net -12V: now also C17.2
- net GND: now also C17.1, C8.1
- net at R8.1: now also C8.2
Other:
- note added: "TDA2050"
- note removed: "1. Wider traces 2oz copper?"
- note removed: "10. Fix -12v D1 slik screen"
- note removed: "11. Move pwr to heat sink, audio in to bottom board"
- note removed: "2. Update heat sink silk screen, get size correct!"
- note removed: "3. C2 & C6 to 10uF"
- note removed: "4. Volume pot, better layout, silk screen"
- note removed: "5. Move R5, heat sink problem"
- note removed: "6. Label amp V gain"
- note removed: "7. speaker wire slik screen correction"
- note removed: "8. Move all the 1000uF caps together."
- note removed: "9. Move pwr jack away from vol pot."
- note removed: "Rev 3 notes"
- moved on the sheet: R14
